File: hw/sch_pcb/UST5BATT18650V01A.kicad_pcb (KiCad board)
At the start: 2 copper layers, 100 x 78 mm, 25 parts, among them J1 SM03B-GHS-TB, J2 SM03B-GHS-TB, X1 TPS63060

Commit message: Edit PCB
Routing:
- net GND: vias 163 -> 171
- added copper zone on B.Cu, net Net-(C1-Pad2)
- added copper zone on B.Cu, net VDD
Changed lines of the file:
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@@
   (via (at 161.393905 100.076) (size 0.8) (drill 0.4) (layers "F.Cu" "B.Cu") (free) (net 1))
   (via (at 118.352455 128.524) (size 0.8) (drill 0.4) (layers "F.Cu" "B.Cu") (free) (net 1))
-  (via (at 153.242815 100.076) (size 0.8) (drill 0.4) (layers "F.Cu" "B.Cu") (free) (net 1))
   (via (at 130.57909 128.524) (size 0.8) (drill 0.4) (layers "F.Cu" "B.Cu") (free) (net 1))
   (via (at 147.193 120.396) (size 0.8) (drill 0.4) (layers "F.Cu" "B.Cu") (free) (net 1))
@@
   (via (at 161.036 120.015) (size 0.8) (drill 0.4) (layers "F.Cu" "B.Cu") (free) (net 1))
   (via (at 147.574 109.22) (size 0.8) (drill 0.4) (layers "F.Cu" "B.Cu") (free) (net 1))
-  (via (at 157.31836 100.076) (size 0.8) (drill 0.4) (layers "F.Cu" "B.Cu") (free) (net 1))
+  (via (at 161.9885 119.126) (size 0.8) (drill 0.4) (layers "F.Cu" "B.Cu") (free) (net 1))
   (via (at 124.714 100.076) (size 0.8) (drill 0.4) (layers "F.Cu" "B.Cu") (free) (net 1))
   (via (at 156.845 123.952) (size 0.8) (drill 0.4) (layers "F.Cu" "B.Cu") (free) (net 1))
   (via (at 147.828 140.208) (size 0.8) (drill 0.4) (layers "F.Cu" "B.Cu") (free) (net 1))
   (via (at 97.155 140.208) (size 0.8) (drill 0.4) (layers "F.Cu" "B.Cu") (free) (net 1))
+  (via (at 148.1455 121.285) (size 0.8) (drill 0.4) (layers "F.Cu" "B.Cu") (free) (net 1))
   (via (at 145.091725 100.076) (size 0.8) (drill 0.4) (layers "F.Cu" "B.Cu") (free) (net 1))
   (via (at 154.178 122.428) (size 0.8) (drill 0.4) (layers "F.Cu" "B.Cu") (free) (net 1))
@@
   (via (at 163.18345 128.524) (size 0.8) (drill 0.4) (layers "F.Cu" "B.Cu") (free) (net 1))
   (via (at 155.321 119.126) (size 0.8) (drill 0.4) (layers "F.Cu" "B.Cu") (free) (net 1))
+  (via (at 150.0505 121.285) (size 0.8) (drill 0.4) (layers "F.Cu" "B.Cu") (free) (net 1))
   (via (at 118.364 140.208) (size 0.8) (drill 0.4) (layers "F.Cu" "B.Cu") (free) (net 1))
   (via (at 171.33455 128.524) (size 0.8) (drill 0.4) (layers "F.Cu" "B.Cu") (free) (net 1))
@@
   (via (at 85.748095 128.524) (size 0.8) (drill 0.4) (layers "F.Cu" "B.Cu") (free) (net 1))
   (via (at 156.21 124.714) (size 0.8) (drill 0.4) (layers "F.Cu" "B.Cu") (free) (net 1))
+  (via (at 162.941 120.015) (size 0.8) (drill 0.4) (layers "F.Cu" "B.Cu") (free) (net 1))
   (via (at 156.337 114.427) (size 0.8) (drill 0.4) (layers "F.Cu" "B.Cu") (free) (net 1))
   (via (at 147.574 107.188) (size 0.8) (drill 0.4) (layers "F.Cu" "B.Cu") (free) (net 1))
   (via (at 154.051 116.84) (size 0.8) (drill 0.4) (layers "F.Cu" "B.Cu") (free) (net 1))
+  (via (at 163.8935 120.015) (size 0.8) (drill 0.4) (layers "F.Cu" "B.Cu") (free) (net 1))
   (via (at 149.16727 100.076) (size 0.8) (drill 0.4) (layers "F.Cu" "B.Cu") (free) (net 1))
   (via (at 157.353 111.379) (size 0.8) (drill 0.4) (layers "F.Cu" "B.Cu") (free) (net 1))
@@
   (via (at 167.59382 70.612) (size 0.8) (drill 0.4) (layers "F.Cu" "B.Cu") (free) (net 1))
   (via (at 110.53618 70.612) (size 0.8) (drill 0.4) (layers "F.Cu" "B.Cu") (free) (net 1))
+  (via (at 149.098 121.285) (size 0.8) (drill 0.4) (layers "F.Cu" "B.Cu") (free) (net 1))
   (via (at 172.339 85.217) (size 0.8) (drill 0.4) (layers "F.Cu" "B.Cu") (free) (net 1))
   (via (at 159.44272 70.612) (size 0.8) (drill 0.4) (layers "F.Cu" "B.Cu") (free) (net 1))
@@
   (via (at 157.353 112.395) (size 0.8) (drill 0.4) (layers "F.Cu" "B.Cu") (free) (net 1))
   (via (at 83.95855 100.076) (size 0.8) (drill 0.4) (layers "F.Cu" "B.Cu") (free) (net 1))
+  (via (at 163.8935 119.126) (size 0.8) (drill 0.4) (layers "F.Cu" "B.Cu") (free) (net 1))
   (via (at 126.503545 128.524) (size 0.8) (drill 0.4) (layers "F.Cu" "B.Cu") (free) (net 1))
   (via (at 132.86509 100.076) (size 0.8) (drill 0.4) (layers "F.Cu" "B.Cu") (free) (net 1))
@@
   (via (at 155.278666 140.208) (size 0.8) (drill 0.4) (layers "F.Cu" "B.Cu") (free) (net 1))
   (via (at 150.0505 120.396) (size 0.8) (drill 0.4) (layers "F.Cu" "B.Cu") (free) (net 1))
+  (via (at 162.941 119.126) (size 0.8) (drill 0.4) (layers "F.Cu" "B.Cu") (free) (net 1))
   (via (at 77.93182 70.612) (size 0.8) (drill 0.4) (layers "F.Cu" "B.Cu") (free) (net 1))
   (via (at 141.01618 100.076) (size 0.8) (drill 0.4) (layers "F.Cu" "B.Cu") (free) (net 1))
+  (via (at 147.193 121.285) (size 0.8) (drill 0.4) (layers "F.Cu" "B.Cu") (free) (net 1))
   (via (at 102.050275 128.524) (size 0.8) (drill 0.4) (layers "F.Cu" "B.Cu") (free) (net 1))
+  (via (at 161.9885 120.015) (size 0.8) (drill 0.4) (layers "F.Cu" "B.Cu") (free) (net 1))
   (via (at 157.353 109.347) (size 0.8) (drill 0.4) (layers "F.Cu" "B.Cu") (free) (net 1))
   (via (at 147.574 113.284) (size 0.8) (drill 0.4) (layers "F.Cu" "B.Cu") (free) (net 1))
@@
   (segment (start 152.9865 126.7585) (end 152.974 126.746) (width 1) (layer "B.Cu") (net 14))
   (segment (start 89.916 136.2225) (end 152.9865 136.2225) (width 1) (layer "B.Cu") (net 14))
-  (segment (start 163.27 92) (end 157.861 97.409) (width 0.5) (layer "B.Cu") (net 15))
-  (segment (start 164.465 83.439) (end 163.27 84.634) (width 0.5) (layer "B.Cu") (net 15))
-  (segment (start 154.305 100.965) (end 154.305 102.952) (width 0.5) (layer "B.Cu") (net 15))
-  (segment (start 157.861 97.409) (end 154.305 100.965) (width 0.5) (layer "B.Cu") (net 15))
-  (segment (start 163.27 84.634) (end 163.27 92) (width 0.5) (layer "B.Cu") (net 15))
-  (segment (start 172.284 92) (end 163.27 92) (width 0.5) (layer "B.Cu") (net 15))
-  (segment (start 168.584 83.439) (end 164.465 83.439) (width 0.5) (layer "B.Cu") (net 15))
+  (segment (start 163.778 84.38) (end 164.719 83.439) (width 0.5) (layer "B.Cu") (net 15))
+  (segment (start 164.719 83.439) (end 168.584 83.439) (width 0.5) (layer "B.Cu") (net 15))
+  (segment (start 163.778 92) (end 172.284 92) (width 0.5) (layer "B.Cu") (net 15))
+  (segment (start 163.778 92) (end 163.778 84.38) (width 0.5) (layer "B.Cu") (net 15))
+  (segment (start 157.607 98.171) (end 163.778 92) (width 0.5) (layer "B.Cu") (net 15))
+  (segment (start 157.099 98.171) (end 157.607 98.171) (width 0.5) (layer "B.Cu") (net 15))
+  (segment (start 154.305 102.952) (end 154.305 100.965) (width 0.5) (layer "B.Cu") (net 15))
+  (segment (start 154.305 100.965) (end 157.099 98.171) (width 0.5) (layer "B.Cu") (net 15))
   (segment (start 149.0745 109.474) (end 149.0745 107.188) (width 0.5) (layer "B.Cu") (net 16))
   (zone (net 1) (net_name "GND") (layers F&B.Cu) (hatch edge 0.508)
     (connect_pads (clearance 0.3))
-    (min_thickness 0.254) (filled_areas_thickness no)
+    (min_thickness 0.2) (filled_areas_thickness no)
     (fill yes (thermal_gap 0.3) (thermal_bridge_width 0.3))
     (polygon
@@
       )
     )
+  )
+  (zone (net 15) (net_name "VDD") (layer "B.Cu") (hatch edge 0.508)
+    (priority 1)
+    (connect_pads yes (clearance 0.3))
+    (min_thickness 0.2) (filled_areas_thickness no)
+    (fill yes (thermal_gap 0.3) (thermal_bridge_width 0.3))
+    (polygon
+      (pts
+        (xy 158.75 103.759)
+        (xy 150.368 103.759)
+        (xy 150.368 97.028)
+        (xy 158.75 97.028)
+      )
+    )
+  )
+  (zone (net 14) (net_name "Net-(C1-Pad2)") (layer "B.Cu") (hatch edge 0.508)
+    (priority 1)
+    (connect_pads yes (clearance 0.2))
+    (min_thickness 0.254) (filled_areas_thickness no)
+    (fill yes (thermal_gap 0.508) (thermal_bridge_width 0.508))
+    (polygon
+      (pts
+        (xy 157.734 136.652)
+        (xy 89.154 136.525)
+        (xy 89.154 134.366)
+        (xy 157.734 134.366)
+      )
+    )
