File: hw/sch_pcb/UST5BATT18650V01.kicad_pcb (KiCad board)
At the start: 2 copper layers, 100 x 78 mm, 32 parts, among them J1 SM04B-GHS-TB, J2 SM03B-GHS-TB, J3 SM03B-GHS-TB, X1 TPS63060

Commit message: Improve silkscreen and readme.
Other:
- board text added: "In the case of charging use only recommended charger."
- board text added: "POWER OUTPUT"
- board text removed: "Chargering"
- board text removed: "POWER OUT"
- board text removed: "Use appropriate charger only."
Changed lines of the file:
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@@
     (property "UST_ID" "5c70984812875079b91f8bbe")
     (attr smd)
-    (fp_text reference "C5" (at -4.318 -0.889) (layer "B.SilkS")
+    (fp_text reference "C5" (at 0 -1.778) (layer "B.SilkS")
       (effects (font (size 1 1) (thickness 0.15)) (justify mirror))
     )
@@
     (property "UST_ID" "")
     (attr smd)
-    (fp_text reference "F4" (at -1.944 3.3 90) (layer "B.SilkS")
+    (fp_text reference "F4" (at 4.826 -0.216 90) (layer "B.SilkS")
       (effects (font (size 1.524 1.524) (thickness 0.3048)) (justify mirror))
     )
@@
     (property "UST_ID" "5c70984412875079b91f8823")
     (attr through_hole)
-    (fp_text reference "L1" (at 0 0 90) (layer "B.SilkS")
+    (fp_text reference "L1" (at -5.334 -8.128 90) (layer "B.SilkS")
       (effects (font (size 1.524 1.524) (thickness 0.3048)) (justify mirror))
     )
@@
     (property "UST_ID" "5c70984612875079b91f89c2")
     (attr smd)
-    (fp_text reference "X1" (at -0.049 2.81 90) (layer "B.SilkS")
+    (fp_text reference "X1" (at 3.253 -2.27 90) (layer "B.SilkS")
       (effects (font (size 1 1) (thickness 0.15)) (justify mirror))
     )
@@
     (property "UST_ID" "612880e51287500165a978de")
     (attr smd)
-    (fp_text reference "J3" (at 0 3.9 90) (layer "B.SilkS")
+    (fp_text reference "J3" (at -5.028 0 90) (layer "B.SilkS")
       (effects (font (size 1 1) (thickness 0.15)) (justify mirror))
     )
@@
     (effects (font (size 1.5 1.5) (thickness 0.2)) (justify left mirror))
   )
-  (gr_text "POWER OUT" (at 165.91 88.04 90) (layer "B.SilkS")
+  (gr_text "POWER OUTPUT" (at 165.862 87.63 90) (layer "B.SilkS")
     (effects (font (size 1.3 1.3) (thickness 0.2)) (justify mirror))
   )
@@
     (effects (font (size 2 2) (thickness 0.3)) (justify mirror))
   )
-  (gr_text "Use appropriate\ncharger only." (at 138.11 118.89 90) (layer "B.SilkS")
+  (gr_text "In the case of charging\nuse only recommended charger." (at 125.476 83.312 90) (layer "B.SilkS")
     (effects (font (size 1.5 1.5) (thickness 0.2)) (justify left mirror))
   )
@@
     (effects (font (size 1.5 1.5) (thickness 0.2)) (justify left mirror))
   )
-  (gr_text "Chargering" (at 133.66 126.94 90) (layer "B.SilkS")
-    (effects (font (size 2 2) (thickness 0.3)) (justify mirror))
-  )
   (gr_text "UST.CZ\nUST5BATT18650V01B" (at 77.47 85.471 90) (layer "F.SilkS")
